Commit message: fix(fr3): cancel timed-out goals, and stop losing the first chunk to discovery
Three review findings on the polyumi_tcp work, each with a check that fails
without the fix.

fr3_moveit_bridge: an execution timeout logged and returned, leaving the goal
running. The caller releases _busy on the way out, so the next chunk planned a
Cartesian path from a start state the arm had already left. Now it cancels and
waits (CANCEL_TIMEOUT_S) for the abort to land before returning; if the cancel
is ignored it says so and names the Desk UI. /polyumi/home made this likely to
bite rather than theoretical: at vscale=0.05 a homing sweep is stretched 20x,
which sits close to HOME_EXECUTE_TIMEOUT_S.

tcp_pivot_test: the first sweep was published without waiting for the bridge's
subscription to match. DDS discovery is asynchronous, so that chunk could
vanish silently and surface as "the arm never moved" — an error whose text
blames execute_arm or an in-flight chunk, i.e. the wrong pane. wait_for_subscriber
covers both first-publishes (arm, and the gripper close when enabled) from run().

tcp_pivot_test: the motion-rate threshold was evaluated between adjacent 50 ms
samples, where 0.01 rad/s is 0.5 mrad — close enough to arm jitter that noise
could latch `moved` and keep resetting the quiet timer, so a finished sweep
would never be detected and would burn the full sweep_timeout_s. It is now
measured against a baseline RATE_WINDOW_S old; drift is still sampled every
period.

Also: main() constructs the node inside the try, so the parameter validation it
already tests for exits cleanly instead of skipping rclpy.shutdown() under a
traceback; and fr3_polyumi.urdf.xacro fails loudly on hand:=false (polyumi_tcp
hangs off fr3_hand) rather than emitting a dangling parent link, using the same
undefined-name trick as its UNSET_* arg defaults.

Co-Authored-By: Claude Opus 5 <noreply@anthropic.com>

File: nuc/description/fr3_polyumi.urdf.xacro (robot description, xacro)
@@ -19,4 +19,14 @@
        are global, so callers set them exactly as they would on fr3.urdf.xacro itself. -->
   <xacro:include filename="$(find franka_description)/robots/fr3/fr3.urdf.xacro" />
+  <!-- polyumi_tcp hangs off ${arm_id}_hand, which fr3.urdf.xacro only creates when hand:=true
+       (its default). With hand:=false the joint below would reference a link that does not exist,
+       and the URDF parser reports that as a dangling parent somewhere in a 400-line generated
+       file. Referencing an undefined name instead fails here, naming the actual problem — the
+       same trick as the UNSET_* arg defaults above, and for the same reason. xacro has no
+       fail/assert, and property values are lazy, so the reference has to sit in an attribute to
+       be evaluated at all. -->
+  <xacro:unless value="$(arg hand)">
+    <link name="${POLYUMI_TCP_NEEDS_hand_true}" />
+  </xacro:unless>
   <link name="polyumi_tcp" />
   <joint name="polyumi_tcp_joint" type="fixed">
